File: sampling design/sampling_design/sampling_design.kicad_sch (KiCad schematic)
At the start: 19 parts, among them U1 LM358, U2 AD708AQ, U3 ESP32-S3-DEVKITC-1-N8R2

Commit message: update schematic sampling design
Parts:
- removed U2: AD708AQ, Q_8_ADI, symbol AD708AQ:AD708AQ
- added BC1: LM2596_Module, symbol Buck_Converter_Module:LM2596_Module
- added C10, C3, C6: 22u, symbol Device:C_US
- added C2: 0.1u, symbol Device:C_US
- added J1: GX Connector Female, symbol Connector:Conn_01x02_Socket
- added J2: GX Connector Male, symbol Connector:Conn_01x02_Pin
- added J3: Microfit Connector Male, symbol Connector:Conn_01x02_Pin
- added J4: Connector Microfit Female, symbol Connector:Conn_01x02_Socket
- added LR1: AMS1117 5V Module, symbol Linear_Voltage_Regulator_Module:AMS1117_5V_Module
- added LR2: AMS1117 3.3V Module, symbol Linear_Voltage_Regulator_Module:AMS1117_3V3_Module
- added R6: 4k7, symbol Device:R
- added R7: 1k2, symbol Device:R
- added U2: OPA2333AID, OPA2333AID:SOIC127P599X175-8N, symbol OPA2333AID:OPA2333AID
- B1: value (none) -> BME280_Module
- M1: value (none) -> MQ4_Module
- R3, R4: value 4.7k -> 4k7
- T1: value (none) -> TGS2620_Module
- T2: value (none) -> TGS2602_Module
- T3: value (none) -> TGS2600_Module
- T4: value (none) -> TGS5042
Connections:
- net 3V3: now also C10.1, C3.1, LR2.3 (OUT+)
- net 5V: now also C6.1, LR1.3 (OUT+), LR2.1 (IN+), R6.1, U2.8 (V+)
- net GND: now also BC1.2 (IN-), BC1.4 (OUT-), C10.2, C2.2, C3.2, C6.2, J4.1 (Pin_1), LR1.2 (IN-), LR1.4 (OUT-), LR2.2 (IN-), LR2.4 (OUT-), R6.2, R7.1, R7.2, U2.3 (+IN_A), U2.4 (V-)
- net TGS5042 Output: now also U2.1 (OUT_A)
- net at C1.1, R2.1, R5.1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: now also U2.2 (-IN_A)
- new net: J1.1 (Pin_1), J3.1 (Pin_1)
- new net: J1.2 (Pin_2), J3.2 (Pin_2)
- new net 12V: BC1.1 (IN+), C2.1, J4.2 (Pin_2)
- new net 6.5V: BC1.3 (OUT+), LR1.1 (IN+)
- new net Adaptor 12V +: J2.2 (Pin_2)
- new net Adaptor 12V -: J2.1 (Pin_1)
- no-connect marks 13 -> 10
Other:
- note added: "Power Connector"
- note added: "Power Distribution"
- moved on the sheet: ADS1, ADS2, C1, R1, R2, R3, R4, R5, RTC1, SD1, U1A, U1C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
